File: connectors.kicad_sch (KiCad schematic)
At the start: 4 parts, among them J1 CONN_01x04_MALE, J2 CONN_01x09_MALE, J3 CONN_01x04_MALE, J4 CONN_MALE_02X03_ODDEVEN

Commit message: Completed Symbol to footprint associations
Parts:
- J1, J3: footprint (none) -> RN_Connectors:J_PTH_CONN_HEADER_MALE_01x04_WUE_61300411121
- J2: footprint (none) -> RN_Connectors:J_PTH_CONN_HEADER_MALE_01x09_WUE_61300911121
- J4: footprint (none) -> RN_Connectors:J_PTH_CONN_HEADER_MALE_02x03_WUE_61300621121
Changed lines of the file:
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@@
     (property "Reference" "J3" (id 0) (at 156.845 93.98 0))
     (property "Value" "CONN_01x04_MALE" (id 1) (at 158.75 96.52 0))
-    (property "Footprint" "" (id 2) (at 156.21 101.6 0)
+    (property "Footprint" "RN_Connectors:J_PTH_CONN_HEADER_MALE_01x04_WUE_61300411121" (id 2) (at 156.21 101.6 0)
       (effects (font (size 1.27 1.27)) hide)
     )
@@
     (property "Reference" "J1" (id 0) (at 132.715 95.25 0))
     (property "Value" "CONN_01x04_MALE" (id 1) (at 132.715 97.79 0))
-    (property "Footprint" "" (id 2) (at 132.08 102.87 0)
+    (property "Footprint" "RN_Connectors:J_PTH_CONN_HEADER_MALE_01x04_WUE_61300411121" (id 2) (at 132.08 102.87 0)
       (effects (font (size 1.27 1.27)) hide)
     )
@@
     (property "Reference" "J4" (id 0) (at 157.48 130.81 0))
     (property "Value" "CONN_MALE_02X03_ODDEVEN" (id 1) (at 157.48 133.35 0))
-    (property "Footprint" "" (id 2) (at 156.21 139.7 0)
+    (property "Footprint" "RN_Connectors:J_PTH_CONN_HEADER_MALE_02x03_WUE_61300621121" (id 2) (at 156.21 139.7 0)
       (effects (font (size 1.27 1.27)) hide)
     )
@@
     (property "Reference" "J2" (id 0) (at 132.715 120.65 0))
     (property "Value" "CONN_01x09_MALE" (id 1) (at 132.715 123.19 0))
-    (property "Footprint" "" (id 2) (at 132.08 135.89 0)
+    (property "Footprint" "RN_Connectors:J_PTH_CONN_HEADER_MALE_01x09_WUE_61300911121" (id 2) (at 132.08 135.89 0)
       (effects (font (size 1.27 1.27)) hide)
     )

Commit message: update schematics
Parts:
- J1, J3: symbol RN_Connectors:CONN_01x04_MALE -> RN_Connectors:CONN_MALE_01x04
- J2: symbol RN_Connectors:CONN_01x09_MALE -> RN_Connectors:CONN_MALE_01x09
Connections:
- net GND: now reaches J3.1
- net GND: now also J1.1, J2.8, J4.6 (Pin_6)
- net Vcc: now reaches J3.2
- net Vcc: now also J1.2, J2.9, J4.2 (Pin_2)
- net RX: now reaches J3.3
- net TX: now reaches J3.4
- net SDA: now reaches J1.3
- net SCK: now reaches J1.4
- net SCK: now also J4.3 (Pin_3)
- net MISO: now reaches J4.1 (Pin_1)
- net MOSI: now reaches J4.4 (Pin_4)
- net RESET: now reaches J4.5 (Pin_5)
- net D2: now reaches J2.1
- net D3: now reaches J2.2
- net D4: now reaches J2.3
- net D5: now reaches J2.4
- net D6: now reaches J2.5
- net D7: now reaches J2.6
- net D8: now reaches J2.7
Other:
- moved on the sheet: J1, J2, J3
Changed lines of the file:
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@@
 (kicad_sch (version 20211123) (generator eeschema)
   (paper "A4")
-  (symbol (lib_id "RN_Connectors:CONN_01x04_MALE") (at 156.21 101.6 0) (unit 1)
+  (hierarchical_label "Vcc" (shape passive) (at 123.19 151.13 0)
+    (effects (font (size 1.27 1.27)) (justify left))
+  )
+  (hierarchical_label "GND" (shape passive) (at 157.48 99.06 0)
+    (effects (font (size 1.27 1.27)) (justify left))
+  )
+  (hierarchical_label "GND" (shape passive) (at 163.83 142.24 0)
+    (effects (font (size 1.27 1.27)) (justify left))
+  )
+  (hierarchical_label "RX" (shape input) (at 157.48 104.14 0)
+    (effects (font (size 1.27 1.27)) (justify left))
+  )
+  (hierarchical_label "D4" (shape bidirectional) (at 123.19 135.89 0)
+    (effects (font (size 1.27 1.27)) (justify left))
+  )
+  (hierarchical_label "SCK" (shape passive) (at 151.13 139.7 180)
+    (effects (font (size 1.27 1.27)) (justify right))
+  )
+  (hierarchical_label "SDA" (shape bidirectional) (at 133.35 105.41 0)
+    (effects (font (size 1.27 1.27)) (justify left))
+  )
+  (hierarchical_label "GND" (shape passive) (at 133.35 100.33 0)
+    (effects (font (size 1.27 1.27)) (justify left))
+  )
+  (hierarchical_label "D6" (shape bidirectional) (at 123.19 140.97 0)
+    (effects (font (size 1.27 1.27)) (justify left))
+  )
+  (hierarchical_label "TX" (shape output) (at 157.48 106.68 0)
+    (effects (font (size 1.27 1.27)) (justify left))
+  )
+  (hierarchical_label "D5" (shape bidirectional) (at 123.19 138.43 0)
+    (effects (font (size 1.27 1.27)) (justify left))
+  )
+  (hierarchical_label "GND" (shape passive) (at 123.19 148.59 0)
+    (effects (font (size 1.27 1.27)) (justify left))
+  )
+  (hierarchical_label "D8" (shape bidirectional) (at 123.19 146.05 0)
+    (effects (font (size 1.27 1.27)) (justify left))
+  )
+  (hierarchical_label "MOSI" (shape input) (at 163.83 139.7 0)
+    (effects (font (size 1.27 1.27)) (justify left))
+  )
+  (hierarchical_label "RESET" (shape passive) (at 151.13 142.24 180)
+    (effects (font (size 1.27 1.27)) (justify right))
+  )
+  (hierarchical_label "D3" (shape bidirectional) (at 123.19 133.35 0)
+    (effects (font (size 1.27 1.27)) (justify left))
+  )
+  (hierarchical_label "D7" (shape bidirectional) (at 123.19 143.51 0)
+    (effects (font (size 1.27 1.27)) (justify left))
+  )
+  (hierarchical_label "MISO" (shape output) (at 151.13 137.16 180)
+    (effects (font (size 1.27 1.27)) (justify right))
+  )
+  (hierarchical_label "Vcc" (shape passive) (at 157.48 101.6 0)
+    (effects (font (size 1.27 1.27)) (justify left))
+  )
+  (hierarchical_label "SCK" (shape passive) (at 133.35 107.95 0)
+    (effects (font (size 1.27 1.27)) (justify left))
+  )
+  (hierarchical_label "Vcc" (shape passive) (at 163.83 137.16 0)
+    (effects (font (size 1.27 1.27)) (justify left))
+  )
+  (hierarchical_label "Vcc" (shape passive) (at 133.35 102.87 0)
+    (effects (font (size 1.27 1.27)) (justify left))
+  )
+  (hierarchical_label "D2" (shape bidirectional) (at 123.19 130.81 0)
+    (effects (font (size 1.27 1.27)) (justify left))
+  )
+  (symbol (lib_id "RN_Connectors:CONN_MALE_01x04") (at 156.21 101.6 0) (unit 1)
     (in_bom yes) (on_board yes)
     (property "Reference" "J3" (id 0) (at 156.845 93.98 0))
     (property "Value" "CONN_01x04_MALE" (id 1) (at 158.75 96.52 0))
-    (property "Footprint" "RN_Connectors:J_PTH_CONN_HEADER_MALE_01x04_WUE_61300411121" (id 2) (at 156.21 101.6 0)
+    (property "Footprint" "RN_Connectors:J_PTH_CONN_HEADER_MALE_01x04_WUE_61300411121" (id 2) (at 157.48 110.49 0)
       (effects (font (size 1.27 1.27)) hide)
     )
-    (property "Datasheet" "~" (id 3) (at 156.21 101.6 0)
+    (property "Datasheet" "~" (id 3) (at 154.94 106.68 0)
       (effects (font (size 1.27 1.27)) hide)
     )
@@
     (pin "4")
   )
-  (symbol (lib_id "RN_Connectors:CONN_01x04_MALE") (at 132.08 102.87 0) (unit 1)
+  (symbol (lib_id "RN_Connectors:CONN_MALE_01x04") (at 132.08 102.87 0) (unit 1)
     (in_bom yes) (on_board yes)
     (property "Reference" "J1" (id 0) (at 132.715 95.25 0))
     (property "Value" "CONN_01x04_MALE" (id 1) (at 132.715 97.79 0))
-    (property "Footprint" "RN_Connectors:J_PTH_CONN_HEADER_MALE_01x04_WUE_61300411121" (id 2) (at 132.08 102.87 0)
+    (property "Footprint" "RN_Connectors:J_PTH_CONN_HEADER_MALE_01x04_WUE_61300411121" (id 2) (at 133.35 111.76 0)
       (effects (font (size 1.27 1.27)) hide)
     )
-    (property "Datasheet" "~" (id 3) (at 132.08 102.87 0)
+    (property "Datasheet" "~" (id 3) (at 130.81 107.95 0)
       (effects (font (size 1.27 1.27)) hide)
     )
@@
     (pin "6")
   )
-  (symbol (lib_id "RN_Connectors:CONN_01x09_MALE") (at 132.08 135.89 0) (unit 1)
+  (symbol (lib_id "RN_Connectors:CONN_MALE_01x09") (at 121.92 133.35 0) (unit 1)
     (in_bom yes) (on_board yes)
-    (property "Reference" "J2" (id 0) (at 132.715 120.65 0))
-    (property "Value" "CONN_01x09_MALE" (id 1) (at 132.715 123.19 0))
-    (property "Footprint" "RN_Connectors:J_PTH_CONN_HEADER_MALE_01x09_WUE_61300911121" (id 2) (at 132.08 135.89 0)
+    (property "Reference" "J2" (id 0) (at 121.92 124.46 0))
+    (property "Value" "CONN_01x09_MALE" (id 1) (at 121.92 127 0))
+    (property "Footprint" "RN_Connectors:J_PTH_CONN_HEADER_MALE_01x09_WUE_61300911121" (id 2) (at 123.19 144.78 0)
       (effects (font (size 1.27 1.27)) hide)
     )
-    (property "Datasheet" "~" (id 3) (at 132.08 135.89 0)
+    (property "Datasheet" "~" (id 3) (at 120.65 140.97 0)
       (effects (font (size 1.27 1.27)) hide)
     )
-    (property "Purpose" "GPIO" (id 4) (at 134.62 149.86 0))
+    (property "Purpose" "GPIO" (id 4) (at 120.65 153.67 0))
     (pin "1")
     (pin "2")
